Commit message: namespace is not working

File: urdf/turtlebot_with_sensor.urdf.xacro (robot description, xacro)
@@ -62,8 +62,8 @@
 </joint> -->
 <joint name="turtlebot_to_base_laser_joint" type="fixed">
-    <origin rpy="0 0 0" xyz="0 0 0.5"/>
+    <origin rpy="0 0 0" xyz="0 0 0.18"/>
     <parent link="base_link"/>
     <child link="base_laser"/>
-    <axis xyz="0 0 0"/>
+    <!-- <axis xyz="0 0 0"/> -->
 </joint>
 </robot>
